Commit message: meshes modified

File: ur_description/urdf/environment.urdf.xacro (robot description, xacro)
@@ -6,5 +6,5 @@
 		<visual>
 			<geometry>
-				<mesh filename="package://ur_description/meshes/environment/feeder_table2.stl" scale="0.01 0.01 0.01"/>
+				<mesh filename="package://ur_description/meshes/environment/table.stl" scale="0.01 0.01 0.01"/>
 			</geometry>
 			<origin xyz="0 0 0"/>
@@ -17,5 +17,5 @@
 		<visual>
 			<geometry>
-				<mesh filename="package://ur_description/meshes/environment/Base_link2.stl"/>
+				<mesh filename="package://ur_description/meshes/environment/mounting.stl"/>
 			</geometry>
 			<origin xyz="0 0 0"/>
